File: fks-0/fks-0.kicad_pcb (KiCad board)
At the start: 2 copper layers, 7 parts, among them J1 Conn_01x15_Socket, J2 Conn_01x15_Socket, M1 Motor_DC, M2 Motor_DC, M3 Motor_DC, M4 Motor_DC

Commit message: add journal
Parts:
- moved M3 160.6 mm to (119.0, 180.1), turned to 180 degrees
- moved M2 145.1 mm to (115.0, 143.9), turned to 0 degrees
- moved M4 114.9 mm to (62.1, 143.9), turned to 180 degrees
- moved J2 57.0 mm to (100.0, 143.9)
- moved J1 56.6 mm to (77.1, 143.9)
- moved BT1 43.9 mm to (90.6, 140.5), turned to 180 degrees
- moved M1 33.9 mm to (58.1, 179.5)
Routing:
- net /GND: track 350.5 -> 155.7 mm
- net /D35: track 0.00 -> 59.3 mm
- net /D34: track 0.00 -> 44.3 mm
- net /D33: track 0.00 -> 27.9 mm
- net /D32: track 0.00 -> 20.4 mm
- net /VIN: track 0.00 -> 10.8 mm
Other:
- board outline added: 70 x 50 mm
