File: fks-0/fks-0.kicad_sch (KiCad schematic)
At the start: 7 parts, among them J1 Conn_01x15_Socket, J2 Conn_01x15_Socket, M1 Motor_DC, M2 Motor_DC, M3 Motor_DC, M4 Motor_DC

Commit message: add journal
Changed lines of the file:
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@@
 	)
 	(junction
-		(at 156.21 87.63)
+		(at 91.44 87.63)
 		(diameter 0)
 		(color 0 0 0 0)
@@
 	(wire
 		(pts
-			(xy 135.89 87.63) (xy 156.21 87.63)
+			(xy 135.89 87.63) (xy 167.64 87.63)
 		)
 		(stroke
@@
 	(wire
 		(pts
-			(xy 156.21 87.63) (xy 167.64 87.63)
-		)
-		(stroke
-			(width 0)
-			(type default)
-		)
-	)
-	(wire
-		(pts
 			(xy 148.59 140.97) (xy 148.59 110.49)
 		)
@@
 	(wire
 		(pts
-			(xy 100.33 87.63) (xy 78.74 87.63)
-		)
-		(stroke
-			(width 0)
-			(type default)
-		)
-	)
-	(wire
-		(pts
-			(xy 156.21 87.63) (xy 156.21 128.27)
+			(xy 100.33 87.63) (xy 91.44 87.63)
+		)
+		(stroke
+			(width 0)
+			(type default)
+		)
+	)
+	(wire
+		(pts
+			(xy 156.21 128.27) (xy 91.44 128.27)
 		)
 		(stroke
@@
 	(wire
 		(pts
-			(xy 156.21 74.93) (xy 156.21 87.63)
-		)
-		(stroke
-			(width 0)
-			(type default)
-		)
-	)
-	(wire
-		(pts
 			(xy 78.74 87.63) (xy 78.74 129.54)
 		)
@@
 	(wire
 		(pts
+			(xy 91.44 74.93) (xy 91.44 87.63)
+		)
+		(stroke
+			(width 0)
+			(type default)
+		)
+	)
+	(wire
+		(pts
 			(xy 78.74 87.63) (xy 78.74 77.47)
 		)
@@
 	(wire
 		(pts
+			(xy 91.44 128.27) (xy 91.44 87.63)
+		)
+		(stroke
+			(width 0)
+			(type default)
+		)
+	)
+	(wire
+		(pts
 			(xy 144.78 142.24) (xy 144.78 113.03)
 		)
@@
 	(wire
 		(pts
+			(xy 91.44 87.63) (xy 78.74 87.63)
+		)
+		(stroke
+			(width 0)
+			(type default)
+		)
+	)
+	(wire
+		(pts
 			(xy 78.74 142.24) (xy 144.78 142.24)
 		)
 		(stroke
+			(width 0)
+			(type default)
+		)
+	)
+	(wire
+		(pts
+			(xy 156.21 74.93) (xy 91.44 74.93)
+		)
+		(stroke
